Commit message: Camera in gazebo

File: src/disp_cv/urdf/camera_desc.urdf.xacro (robot description, xacro)
@@ -1,7 +1,8 @@
 <?xml version="1.0" ?>
 <robot xmlns:xacro="http://ros.org/wiki/xacro">
+ <xacro:macro name="camera_xtion">
   <link name="camera_asus">
       <collision>
-        <origin xyz="0 0 0" rpy="0 0 0"/>
+        <origin xyz="0 0 0.03" rpy="0 0 0"/>
         <geometry>
             <box size="0.2 0.06 0.06" />
@@ -9,7 +10,7 @@
       </collision>
       <visual>
-        <origin xyz="0 0 0" rpy="0 0 0"/>
+        <origin xyz="0 0 0.03" rpy="0 0 0"/>
         <geometry>
-            <box size="0.2 0.06 0.06" />
+            <box size="0.06 0.2 0.06" />
         </geometry>
         <material name="red_c">
@@ -23,3 +24,4 @@
       </inertial>
   </link>
+</xacro:macro>
 </robot>

File: src/disp_cv/urdf/env_model.urdf.xacro (robot description, xacro)
@@ -4,20 +4,124 @@
   <xacro:include filename="$(find disp_cv)/urdf/camera_desc.urdf.xacro"/>
   <xacro:include filename="$(find ur_description)/urdf/ur5.urdf.xacro"/>
-  <xacro:ur5_robot prefix="ur5_" joint_limited="true"/>
+  <xacro:include filename="$(find disp_cv)/urdf/common_gazebo.gazebo.xacro" />
+  <xacro:ur5_robot prefix="" joint_limited="true"/>
+  <xacro:support/>
+  <xacro:camera_xtion/>
   <joint name="camera_to_camera_holder" type="fixed">
     <parent link="camera_holder"/>
     <child link="camera_asus"/>
-    <origin xyz="0 0.15 0.625" rpy="0 0 0"/>
+    <origin xyz="0.20 0.0475 0.375" rpy="0 0 0"/>
   </joint>
-  <joint name="ur5_robot_to_mount" type="fixed">
-    <parent link="mount"/>
-    <child link="ur5_base_link"/>
-    <origin xyz="0 0 0.85" rpy="0 0 0"/>
-  </joint>
-  <link name="world" />
- <joint name="world_joint" type="fixed">
-   <parent link="world" />
-   <child link = "base" />
-   <origin xyz="0.0 0.0 0.0" rpy="0.0 0.0 0.0" />
- </joint>
+<joint name="ur5_robot_to_mount" type="fixed">
+  <parent link="mount"/>
+  <child link="base_link"/>
+  <origin xyz="0 0 0.60" rpy="0 0 0"/>
+</joint>
+<link name="world" />
+<joint name="world_joint" type="revolute">
+  <parent link="world" />
+  <child link = "base_support" />
+  <origin xyz="0.0 0.0 0.0" rpy="0.0 0.0 0.0" />
+  <axis xyz="0 0 1"/>
+  <limit lower="${-2.0 * pi}" upper="${2.0 * pi}" effort="150.0" velocity="3.15"/>
+</joint>
+<gazebo reference="camera_asus">
+  <mu1>0.2</mu1>
+  <mu2>0.2</mu2>
+  <material>Gazebo/Black</material>
+</gazebo>
+<gazebo reference="mount">
+  <mu1>0.2</mu1>
+  <mu2>0.2</mu2>
+  <material>Gazebo/Grey</material>
+</gazebo>
+<gazebo reference="camera_holder">
+  <mu1>0.2</mu1>
+  <mu2>0.2</mu2>
+  <material>Gazebo/Grey</material>
+</gazebo>
+<gazebo reference="camera_asus">
+    <sensor name="camera" type="depth">
+       <camera>
+         <horizontal_fov>1.047</horizontal_fov>
+         <image>
+           <width>640</width>
+           <height>480</height>
+         </image>
+         <clip>
+           <near>0.3</near>
+           <far>20</far>
+         </clip>
+       </camera>
+       <always_on>1</always_on>
+       <update_rate>30</update_rate>
+       <visualize>true</visualize>
+       <plugin name="camera_plugin" filename="libgazebo_ros_openni_kinect.so">
+                 <baseline>0.2</baseline>
+                 <alwaysOn>true</alwaysOn>
+                 <!-- Keep this zero, update_rate in the parent <sensor> tag
+                   will control the frame rate. -->
+                 <updateRate>0.0</updateRate>
+                 <cameraName>camera_ir</cameraName>
+                 <imageTopicName>/gaz_camera/depth/image_raw</imageTopicName>
+                 <cameraInfoTopicName>/gaz_camera/depth/camera_info</cameraInfoTopicName>
+                 <depthImageTopicName>/gaz_camera/depth/image_raw</depthImageTopicName>
+                 <depthImageInfoTopicName>/gaz_camera/depth/camera_info</depthImageInfoTopicName>
+                 <pointCloudTopicName>/gaz_camera/depth/points</pointCloudTopicName>
+                 <frameName>camera_rgb_optical_frame</frameName>
+                 <pointCloudCutoff>0.3</pointCloudCutoff>
+                 <distortionK1>0</distortionK1>
+                 <distortionK2>0</distortionK2>
+                 <distortionK3>0</distortionK3>
+                 <distortionT1>0</distortionT1>
+                 <distortionT2>0</distortionT2>
+                 <CxPrime>0</CxPrime>
+                 <Cx>0</Cx>
+                 <Cy>0</Cy>
+                 <focalLength>0</focalLength>
+                 <hackBaseline>0</hackBaseline>
+        </plugin>
+     </sensor>
+    </gazebo>
+    <gazebo reference="camera_asus">
+        <sensor name="camera" type="camera">
+           <camera>
+             <horizontal_fov>1.047</horizontal_fov>
+             <image>
+               <width>640</width>
+               <height>480</height>
+               <format>R8G8B8</format>
+             </image>
+             <clip>
+               <near>0.02</near>
+               <far>300</far>
+             </clip>
+           </camera>
+           <always_on>1</always_on>
+           <update_rate>30</update_rate>
+           <visualize>true</visualize>
+           <noise>
+                   <type>gaussian</type>
+                   <!-- Noise is sampled independently per pixel on each frame.
+                        That pixel's noise value is added to each of its color
+                        channels, which at that point lie in the range [0,1]. -->
+                   <mean>0.0</mean>
+                   <stddev>0.007</stddev>
+                 </noise>
+           <plugin name="camera_controller" filename="libgazebo_ros_camera.so">
+           <alwaysOn>true</alwaysOn>
+           <updateRate>0.0</updateRate>
+           <cameraName>ur5/camera1</cameraName>
+           <imageTopicName>gaz_camera/image_raw</imageTopicName>
+           <cameraInfoTopicName>camera_info</cameraInfoTopicName>
+           <frameName>camera_rgb_optical_frame</frameName>
+           <hackBaseline>0.07</hackBaseline>
+           <distortionK1>0.0</distortionK1>
+           <distortionK2>0.0</distortionK2>
+           <distortionK3>0.0</distortionK3>
+           <distortionT1>0.0</distortionT1>
+           <distortionT2>0.0</distortionT2>
+         </plugin>
+         </sensor>
+        </gazebo>
 </robot>

File: src/disp_cv/urdf/table_info.urdf.xacro (robot description, xacro)
@@ -1,22 +1,31 @@
 <?xml version="1.0" ?>
 <robot xmlns:xacro="http://ros.org/wiki/xacro">
-  <link name="base">
+<xacro:macro name="support">
+<material name ="custom">
+      <color rgba="0.3 0.1 0.3 1"/>
+      <ambient> .175 .175 .175  1.0</ambient>
+      <diffuse> .175 .175 .175  1.0</diffuse>
+      <specular> .175 .175 .175 1.000000 1.500000</specular>
+    </material>
+  <link name="base_support">
      <inertial>
           <mass value="10" />
-          <origin xyz="0 0 0" rpy="0 0 0"/>
-          <inertia ixx="0.0833" iyy="0.0833" izz="0.0633" ixy="0" ixz="0" iyz="0"/>
+          <origin xyz="0 0.0 0.175" rpy="0 0 0"/>
+          <inertia ixx="0.58541667" iyy="0.58541667" izz="1.066667" ixy="0" ixz="0" iyz="0"/>
      </inertial>
      <visual>
-       <origin xyz="0 0 0" rpy="0 0 0"/>
+       <origin xyz="0 0.0 0.175" rpy="0 0 0"/>
        <geometry>
             <box size="0.8 0.8 0.25 "/>
        </geometry>
-       <material name="blue_c">
+     <!--  <material>
          <color rgba="0.2 0 1 0.9"/>
-       </material>
+       </material>-->
+       <material name="custom"/>
      </visual>
      <collision>
+        <origin xyz="0 0.0 0.175" rpy="0 0 0"/>
         <geometry>
-            <box size="0.5 0.5 0.25"/>
+            <box size="0.8 0.8 0.25"/>
         </geometry>
      </collision>
@@ -25,17 +34,17 @@
   <inertial>
        <mass value="4" />
-      <origin xyz="0 0 0" rpy="0 0 0"/>
-      <inertia ixx="0.0833" iyy="0.0833" izz="0.0633" ixy="0" ixz="0" iyz="0"/>
+      <inertia ixx="0.06375" iyy="0.114375" izz="0.084375" ixy="0" ixz="0" iyz="0"/>
   </inertial>
   <visual>
-      <origin xyz="0 0.0375 0" rpy="0 0 0"/>
+      <origin xyz="0 0.0475 0.1875" rpy="0 0 0"/>
       <geometry>
           <box size="0.45 0.225 0.375"/>
       </geometry>
-      <material name="green_c">
+     <!-- <material >
           <color rgba="0 1 0.1 0.5"/>
-      </material>
+      </material>-->
   </visual>
   <collision>
+      <origin xyz="0 0.0475 0.1875" rpy="0 0 0"/>
       <geometry>
            <box size="0.45 0.225 0.375"/>
@@ -43,37 +52,43 @@
   </collision>
 </link>
+<joint name="base_to_camera_holder" type="fixed">
+   <parent link="base_support"/>
+   <child link="camera_holder"/>
+   <origin xyz="0 0.15 0.30" rpy="0 0 0"/>
+   <inertial>
+   <mass value="0.001"/>
+   <inertia ixx="5.1458e-5" iyy="5.1458e-5" izz="5.1458e-5" ixy="0" ixz="0" iyz="0"/>
+   </inertial>
+</joint>
   <link name="mount">
      <inertial>
         <mass value="7" />
-        <origin xyz="0 0 0" rpy="0 0 0"/>
-        <inertia ixx="0.0833" iyy="0.0833" izz="0.0633" ixy="0" ixz="0" iyz="0"/>
+        <inertia ixx="0.21984" iyy="0.21984" izz="0.0098398" ixy="0" ixz="0" iyz="0"/>
      </inertial>
      <visual>
-       <origin xyz="0 0 0" rpy="0 0 0"/>
+       <origin xyz="0 0 0.30" rpy="0 0 0"/>
        <geometry>
           <cylinder length="0.60" radius= "0.075"/>
        </geometry>
-       <material name="red_c">
+      <!-- <material >
         <color rgba="1 0.2 0 0.9"/>
-       </material>
+       </material> -->
      </visual>
+     <collision>
+     <origin xyz="0 0 0.30" rpy="0 0 0"/>
+         <geometry>
+              <cylinder length="0.60" radius="0.075"/>
+         </geometry>
+     </collision>
    </link>
-  <joint name="base_to_mount" type="fixed">
-    <parent link="base"/>
-    <child link="mount"/>
-    <origin xyz="0 0 0.25" rpy="0 0 0"/>
-    <inertial>
-    <mass value="1.0"/>
-    <inertia ixx="5.1458e-5" iyy="5.1458e-5" izz="5.1458e-5" ixy="0" ixz="0" iyz="0"/>
-    </inertial>
-  </joint>
- <joint name="base_to_camera_holder" type="fixed">
-    <parent link="base"/>
-    <child link="camera_holder"/>
-    <origin xyz="0 0.15 0.25" rpy="0 0 0"/>
-    <inertial>
-    <mass value="1.0"/>
-    <inertia ixx="5.1458e-5" iyy="5.1458e-5" izz="5.1458e-5" ixy="0" ixz="0" iyz="0"/>
-    </inertial>
- </joint>
+   <joint name="base_to_mount" type="fixed">
+     <parent link="base_support"/>
+     <child link="mount"/>
+     <origin xyz="0 0 0.30" rpy="0 0 0"/>
+     <inertial>
+     <mass value="0.001"/>
+     <inertia ixx="5.1458e-5" iyy="5.1458e-5" izz="5.1458e-5" ixy="0" ixz="0" iyz="0"/>
+     </inertial>
+   </joint>
+  </xacro:macro>
 </robot>
