Commit message: Ur modifications

File: src/disp_cv/urdf/common_gazebo.gazebo.xacro (robot description, xacro)
@@ -1,9 +1,10 @@
 <?xml version="1.0"?>
 <robot xmlns:xacro="http://ros.org/wiki/xacro">
-  <gazebo>
-    <plugin name="ros_control" filename="libgazebo_ros_control.so">
-      <!--robotNamespace>/</robotNamespace-->
-      <!--robotSimType>gazebo_ros_control/DefaultRobotHWSim</robotSimType-->
+<gazebo>
+    <plugin name="gazebo_ros_control" filename="libgazebo_ros_control.so">
+      <robotNamespace>/ur5robot</robotNamespace>
+      <robotSimType>gazebo_ros_control/DefaultRobotHWSim</robotSimType>
     </plugin>
+</gazebo>
 <!--
     <plugin name="camera_plugin" filename="libgazebo_ros_openni_kinect.so">
@@ -47,4 +48,3 @@
     </plugin>
 -->
-  </gazebo>
 </robot>

File: src/disp_cv/urdf/env_model.urdf.xacro (robot description, xacro)
@@ -1,15 +1,25 @@
 <?xml version="1.0" ?>
-<robot name="ur5_robot_and env" xmlns:xacro="http://ros.org/wiki/xacro">
+<robot name="ur5robot" xmlns:xacro="http://ros.org/wiki/xacro">
   <xacro:include filename="$(find disp_cv)/urdf/table_info.urdf.xacro"/>
   <xacro:include filename="$(find disp_cv)/urdf/camera_desc.urdf.xacro"/>
   <xacro:include filename="$(find ur_description)/urdf/ur5.urdf.xacro"/>
   <xacro:include filename="$(find disp_cv)/urdf/common_gazebo.gazebo.xacro" />
-  <xacro:ur5_robot prefix="" joint_limited="true"/>
+  <xacro:include filename="$(find disp_cv)/urdf/sensor_def.gazebo.xacro"/>
+  <xacro:ur5_robot prefix="" joint_limited="true"
+    shoulder_pan_lower_limit="${-pi}" shoulder_pan_upper_limit="${pi}"
+    shoulder_lift_lower_limit="${-pi}" shoulder_lift_upper_limit="${pi}"
+    elbow_joint_lower_limit="${-pi}" elbow_joint_upper_limit="${pi}"
+    wrist_1_lower_limit="${-pi}" wrist_1_upper_limit="${pi}"
+    wrist_2_lower_limit="${-pi}" wrist_2_upper_limit="${pi}"
+    wrist_3_lower_limit="${-pi}" wrist_3_upper_limit="${pi}"
+  />
   <xacro:support/>
   <xacro:camera_xtion/>
-  <joint name="camera_to_camera_holder" type="fixed">
+  <joint name="camera_to_camera_holder" type="revolute">
     <parent link="camera_holder"/>
     <child link="camera_asus"/>
     <origin xyz="0.20 0.0475 0.375" rpy="0 0 0"/>
+    <axis xyz="0 0 1"/>
+    <limit lower="${-2.0 * pi}" upper="${2.0 * pi}" effort="150.0" velocity="3.15"/>
   </joint>
 <joint name="ur5_robot_to_mount" type="fixed">
@@ -19,109 +29,18 @@
 </joint>
 <link name="world" />
-<joint name="world_joint" type="revolute">
+<joint name="world_joint" type="fixed">
   <parent link="world" />
   <child link = "base_support" />
   <origin xyz="0.0 0.0 0.0" rpy="0.0 0.0 0.0" />
-  <axis xyz="0 0 1"/>
-  <limit lower="${-2.0 * pi}" upper="${2.0 * pi}" effort="150.0" velocity="3.15"/>
 </joint>
-<gazebo reference="camera_asus">
-  <mu1>0.2</mu1>
-  <mu2>0.2</mu2>
-  <material>Gazebo/Black</material>
-</gazebo>
-<gazebo reference="mount">
-  <mu1>0.2</mu1>
-  <mu2>0.2</mu2>
-  <material>Gazebo/Grey</material>
-</gazebo>
-<gazebo reference="camera_holder">
-  <mu1>0.2</mu1>
-  <mu2>0.2</mu2>
-  <material>Gazebo/Grey</material>
-</gazebo>
-<gazebo reference="camera_asus">
-    <sensor name="camera" type="depth">
-       <camera>
-         <horizontal_fov>1.047</horizontal_fov>
-         <image>
-           <width>640</width>
-           <height>480</height>
-         </image>
-         <clip>
-           <near>0.3</near>
-           <far>20</far>
-         </clip>
-       </camera>
-       <always_on>1</always_on>
-       <update_rate>30</update_rate>
-       <visualize>true</visualize>
-       <plugin name="camera_plugin" filename="libgazebo_ros_openni_kinect.so">
-                 <baseline>0.2</baseline>
-                 <alwaysOn>true</alwaysOn>
-                 <!-- Keep this zero, update_rate in the parent <sensor> tag
-                   will control the frame rate. -->
-                 <updateRate>0.0</updateRate>
-                 <cameraName>camera_ir</cameraName>
-                 <imageTopicName>/gaz_camera/depth/image_raw</imageTopicName>
-                 <cameraInfoTopicName>/gaz_camera/depth/camera_info</cameraInfoTopicName>
-                 <depthImageTopicName>/gaz_camera/depth/image_raw</depthImageTopicName>
-                 <depthImageInfoTopicName>/gaz_camera/depth/camera_info</depthImageInfoTopicName>
-                 <pointCloudTopicName>/gaz_camera/depth/points</pointCloudTopicName>
-                 <frameName>camera_rgb_optical_frame</frameName>
-                 <pointCloudCutoff>0.3</pointCloudCutoff>
-                 <distortionK1>0</distortionK1>
-                 <distortionK2>0</distortionK2>
-                 <distortionK3>0</distortionK3>
-                 <distortionT1>0</distortionT1>
-                 <distortionT2>0</distortionT2>
-                 <CxPrime>0</CxPrime>
-                 <Cx>0</Cx>
-                 <Cy>0</Cy>
-                 <focalLength>0</focalLength>
-                 <hackBaseline>0</hackBaseline>
-        </plugin>
-     </sensor>
-    </gazebo>
-    <gazebo reference="camera_asus">
-        <sensor name="camera" type="camera">
-           <camera>
-             <horizontal_fov>1.047</horizontal_fov>
-             <image>
-               <width>640</width>
-               <height>480</height>
-               <format>R8G8B8</format>
-             </image>
-             <clip>
-               <near>0.02</near>
-               <far>300</far>
-             </clip>
-           </camera>
-           <always_on>1</always_on>
-           <update_rate>30</update_rate>
-           <visualize>true</visualize>
-           <noise>
-                   <type>gaussian</type>
-                   <!-- Noise is sampled independently per pixel on each frame.
-                        That pixel's noise value is added to each of its color
-                        channels, which at that point lie in the range [0,1]. -->
-                   <mean>0.0</mean>
-                   <stddev>0.007</stddev>
-                 </noise>
-           <plugin name="camera_controller" filename="libgazebo_ros_camera.so">
-           <alwaysOn>true</alwaysOn>
-           <updateRate>0.0</updateRate>
-           <cameraName>ur5/camera1</cameraName>
-           <imageTopicName>gaz_camera/image_raw</imageTopicName>
-           <cameraInfoTopicName>camera_info</cameraInfoTopicName>
-           <frameName>camera_rgb_optical_frame</frameName>
-           <hackBaseline>0.07</hackBaseline>
-           <distortionK1>0.0</distortionK1>
-           <distortionK2>0.0</distortionK2>
-           <distortionK3>0.0</distortionK3>
-           <distortionT1>0.0</distortionT1>
-           <distortionT2>0.0</distortionT2>
-         </plugin>
-         </sensor>
-        </gazebo>
+<transmission name="camera_move">
+<type>transmission_interface/SimpleTransmission</type>
+<joint name="camera_to_camera_holder">
+    <hardwareInterface>hardware_interface/EffortJointInterface</hardwareInterface>
+</joint>
+<actuator name="motor1">
+    <hardwareInterface>hardware_interface/EffortJointInterface</hardwareInterface>
+    <mechanicalReduction>1</mechanicalReduction>
+</actuator>
+</transmission>
 </robot>
